File: Hardware/Digital Clock PCB 2.0 Module Based.kicad_pcb (KiCad board)
At the start: 2 copper layers, 124.5 x 46 mm, 77 parts, among them J1 USB_C_Receptacle_USB2.0, J2 Conn_01x04, J3 Conn_01x04, Q1 C15127, Q2 C8545, SW1 SW_Push, SW2 SW_Push, U1 ESP32-S2-SOLO-2, U10 SBC18-11SURKCGKWA, U2 AMS1117-3.3, U3 74LS47, U4 74LS47, U5 SBC18-11SURKCGKWA, U6 SBC18-11SURKCGKWA, U7 74LS47, U8 74LS47, U9 SBC18-11SURKCGKWA

Commit message: Final revision for this run
Parts:
- removed C8, C9: C, Capacitor_SMD:C_0805_2012Metric
- removed Q1: C15127, Package_TO_SOT_SMD:SOT-23
- removed Q2: C8545, Package_TO_SOT_SMD:SOT-23
- removed R10, R11, R12, R29, R30, R31, R32, R33, R34, R9: R, Resistor_SMD:R_0603_1608Metric
- removed R4, R5, R6: 47k, Resistor_SMD:R_0805_2012Metric
- removed U1: ESP32-S2-SOLO-2, RF_Module:ESP32-S3-WROOM-1
- removed U4, U7, U8: 74LS47, Package_SO:SOIC-16_4.55x10.3mm_P1.27mm
- added TP1: CHAIN, TestPoint:TestPoint_Pad_D1.5mm, F.Cu at (205.2, 98.2)
- added U11: 74HC595, Package_SO:SOIC-16_3.9x9.9mm_P1.27mm, F.Cu at (235.8, 103.3)
- added U12: 74HC595, Package_SO:SOIC-16_3.9x9.9mm_P1.27mm, F.Cu at (224.2, 103.3)
- added U13: 74HC595, Package_SO:SOIC-16_3.9x9.9mm_P1.27mm, F.Cu at (200.8, 103.3)
- added U14: 74HC595, Package_SO:SOIC-16_3.9x9.9mm_P1.27mm, F.Cu at (212.5, 103.3)
- C6: value C -> 22u; footprint Capacitor_SMD:C_0805_2012Metric -> Capacitor_SMD:C_0603_1608Metric
- C7: value C -> 100n; footprint Capacitor_SMD:C_0805_2012Metric -> Capacitor_SMD:C_0603_1608Metric
- R7, R8: value R -> 4k7
- SW1, SW2: footprint Ian's Custom Components:5.2mm_Tactile_Push_Button -> Button_Switch_SMD:SW_SPST_SKQG_WithStem
- U10, U5, U6, U9: value SBC18-11SURKCGKWA -> FJ15101BH
- U3: value 74LS47 -> ESP32-S3-MINI-1; footprint Package_SO:SOIC-16_4.55x10.3mm_P1.27mm -> RF_Module:ESP32-S2-MINI-1
- moved U3 29.6 mm to (260.0, 103.4), turned to -90 degrees
- moved C6 25.3 mm to (262.5, 93.0), turned to 0 degrees
- moved C7 23.6 mm to (262.5, 94.5), turned to 0 degrees
- moved R8 18.1 mm to (211.5, 115.0)
- moved R7 17.8 mm to (211.5, 113.2)
- moved J3 13.9 mm to (250.2, 115.8)
- moved C5 5.95 mm to (208.0, 115.8), turned to 180 degrees
- moved J2 4.93 mm to (261.4, 115.8)
- moved R3 3.55 mm to (259.5, 93.0)
- moved C3 3.40 mm to (259.5, 94.5)
- moved C4 0.99 mm to (205.4, 114.1)
Connections:
- C6 pad 1: VBUS -> +3V3
- C7 pad 1: VBUS -> +3V3
- J2 pad 1: VBUS -> +3V3
- R13 pad 1: Net-(U3-a) -> Net-(U11-QA)
- R14 pad 1: Net-(U3-b) -> Net-(U11-QB)
- R15 pad 1: Net-(U3-c) -> Net-(U11-QC)
- R16 pad 1: Net-(U3-d) -> Net-(U11-QD)
- R17 pad 1: Net-(U3-e) -> Net-(U11-QE)
- R18 pad 1: Net-(U3-f) -> Net-(U11-QF)
- R19 pad 1: Net-(U3-g) -> Net-(U11-QG)
- R20 pad 1: IO38 -> IO35
- R28 pad 1: IO37 -> IO38
- R42 pad 1: IO35 -> IO36
- R50 pad 1: IO36 -> IO37
- R7 pad 1: GND -> SCL
- R7 pad 2: Net-(U3-LT) -> +3V3
- R8 pad 1: GND -> SDA
- R8 pad 2: Net-(U3-BI) -> +3V3
- SW1 pad 1: Net-(U1-IO0) -> BOOT
- U10 pad 1: CC -> VBUS
- U10 pad 5: CC -> VBUS
- U3 pad 1: B4 -> GND
- U3 pad 10: Net-(U3-d) -> unconnected-(U3-IO6-Pad10)
- U3 pad 11: Net-(U3-c) -> unconnected-(U3-IO7-Pad11)
- U3 pad 12: Net-(U3-b) -> unconnected-(U3-IO8-Pad12)
- U3 pad 13: Net-(U3-a) -> ~{Brightness}
- U3 pad 14: Net-(U3-g) -> unconnected-(U3-IO10-Pad14)
- U3 pad 15: Net-(U3-f) -> Latch
- U3 pad 16: +3V3 -> unconnected-(U3-IO12-Pad16)
- U3 pad 2: C4 -> GND
- U3 pad 3: Net-(U3-LT) -> +3V3
- U3 pad 4: Net-(U3-BI) -> unconnected-(U3-IO0-Pad4)
- U3 pad 5: Net-(U3-RBI) -> unconnected-(U3-IO1-Pad5)
- U3 pad 6: D4 -> BOOT
- U3 pad 7: A4 -> TIME_DATA
- U3 pad 8: GND -> unconnected-(U3-IO4-Pad8)
- U3 pad 9: Net-(U3-e) -> unconnected-(U3-IO5-Pad9)
- U5 pad 1: CC -> VBUS
- U5 pad 5: CC -> VBUS
- U6 pad 1: CC -> VBUS
- U6 pad 5: CC -> VBUS
- U9 pad 1: CC -> VBUS
- U9 pad 5: CC -> VBUS
Routing:
- net +3V3: track 281.5 -> 161.5 mm, vias 17 -> 7
- net CC: track 110.6 -> 0.00 mm
- net VBUS: track 143.4 -> 248.2 mm, vias 4 -> 10
- net B1: track 103.6 -> 0.00 mm, vias 2 -> 0
- net D1: track 102.5 -> 0.00 mm, vias 2 -> 0
- net C1: track 102.2 -> 0.00 mm, vias 2 -> 0
- net A1: track 101.5 -> 0.00 mm, vias 2 -> 0
- net IO38: track 31.5 -> 115.7 mm
- net B2: track 77.2 -> 0.00 mm, vias 2 -> 0
- net D2: track 76.7 -> 0.00 mm, vias 2 -> 0
- net C2: track 76.2 -> 0.00 mm, vias 2 -> 0
- net A2: track 75.6 -> 0.00 mm, vias 2 -> 0
- net Net-(U1-IO0): track 73.8 -> 0.00 mm, vias 2 -> 0
- net IO35: track 99.3 -> 32.2 mm, vias 4 -> 2
- net Latch: track 0.00 -> 62.6 mm, vias 0 -> 5
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Other:
- board text added: "RedShift"
- board text removed: "EEAN"
- board text removed: "PASSWD: MinesBigger"
- board text removed: "SSID: NiceClock"
- board text removed: "http://NiceClock"
